File: hardware/ZRADTri/ZRADTri.kicad_sch (KiCad schematic)
At the start: 62 parts, among them J1 Conn_Coaxial, J2 Qwiic_RA, J3 Conn_Coaxial, J4 Conn_02x05_Counter_Clockwise, J5 Conn_01x02, J6 Conn_01x05, J7 Conn_01x05, J8 USB_C_Receptacle_USB2.0_16P, SW1 PTS810, SW2 PTS810, U1 T32CZ20B20GQ40, U2 AP2127K-3.3, U3 CP2102N-Axx-xQFN24, Y1 39MHz 10ppm

Commit message: initial Trident PCB layout
Parts:
- C15: footprint Capacitor_SMD:C_0805_2012Metric -> Capacitor_SMD:C_0603_1608Metric
- U1: footprint (none) -> Package_DFN_QFN:TQFN-40-1EP_5x5mm_P0.4mm_EP3.5x3.5mm_ThermalVias
Connections:
- net GP06: now reaches U1.31 (GP06)
- net GP06: now also J7.3 (Pin_3)
- net GP00: no longer names the net of U1.35 (GP00)
- net GP00: no longer J7.3 (Pin_3)
Changed lines of the file:
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@@
 	)
 	(no_connect
-		(at 148.59 121.92)
+		(at 148.59 109.22)
 	)
 	(no_connect
@@
 	(wire
 		(pts
-			(xy 129.54 109.22) (xy 148.59 109.22)
-		)
-		(stroke
-			(width 0)
-			(type default)
-		)
-	)
-	(wire
-		(pts
 			(xy 194.31 116.84) (xy 213.36 116.84)
 		)
@@
 	(wire
 		(pts
+			(xy 129.54 121.92) (xy 148.59 121.92)
+		)
+		(stroke
+			(width 0)
+			(type default)
+		)
+	)
+	(wire
+		(pts
 			(xy 247.65 110.49) (xy 248.92 110.49)
 		)
@@
 		)
 	)
-	(label "GP00"
-		(at 135.89 109.22 0)
+	(label "GP06"
+		(at 138.43 121.92 0)
 		(effects
 			(font
@@
 		)
 	)
-	(label "GP00"
+	(label "GP06"
 		(at 36.83 115.57 0)
 		(effects
@@
 			)
 		)
-		(property "Footprint" ""
+		(property "Footprint" "Package_DFN_QFN:TQFN-40-1EP_5x5mm_P0.4mm_EP3.5x3.5mm_ThermalVias"
 			(at 173.99 156.21 0)
 			(effects
@@
 			)
 		)
-		(property "Description" "ARM M33 SubGHz Radio +20dBm 1MB Flash 288KRAM Z-Wave QFN-40"
+		(property "Description" "ARM,M33,SubGHz Radio,+20dBm,1MB,Flash,288KRAM,Z-Wave,QFN-40"
 			(at 172.466 118.11 0)
 			(effects
@@
 			)
 		)
-		(property "Footprint" "Capacitor_SMD:C_0805_2012Metric"
+		(property "Footprint" "Capacitor_SMD:C_0603_1608Metric"
 			(at 133.35 95.25 0)
 			(effects

Commit message: ZRADTri Trident IoT PCB rev A complete
Parts:
- added NE1: 27,-77, MountingHole:MountingHole_2.7mm, symbol Mechanical:MountingHole
- added NW1: 7,-77, MountingHole:MountingHole_2.7mm, symbol Mechanical:MountingHole
- added SE1: 27,-17, MountingHole:MountingHole_2.7mm, symbol Mechanical:MountingHole
- added SW3: 7,-17, MountingHole:MountingHole_2.7mm, symbol Mechanical:MountingHole
- J4: footprint (none) -> Connector:Tag-Connect_TC2050-IDC-NL_2x05_P1.27mm_Vertical
- renumbered C25 to C10, C14 to C11, C11 to C12, C7 to C13, C24 to C14, C23 to C15, C15 to C16, C22 to C17, C13 to C18, C27 to C19, C9 to C2, C26 to C20, C17 to C21, C16 to C22, C18 to C23, C21 to C24, C19 to C25, C20 to C26, C4 to C3, C2 to C4, C3 to C5, C8 to C6, C6 to C7, C5 to C8, C12 to C9, L4 to L1, L3 to L2, L2 to L3, L1 to L4, L6 to L5, L9 to L6, L5 to L7, L7 to L8, L8 to L9, R2 to R1, R5 to R10, R1 to R2, R6 to R5, R7 to R6, R8 to R7, R9 to R8, R10 to R9
Other:
- note added: "Mounting Holes"

Commit message: Updated ZRADTri BOM and schematic with minor changes for Rev A
Parts:
- C10: value 100NF -> 100N
- C13: value 100PF -> 120PF
- C16: footprint Capacitor_SMD:C_0603_1608Metric -> Capacitor_SMD:C_0805_2012Metric
- C20: value 10UF -> 4U7
- L2: value 12N -> 12NH
- L3: value 8N5 -> 8.5NH
- L4, L6: value 27UH -> 27NH
- L5, L7: value 47UH -> 47NH
- L8: value 4U7 -> 4.7UH
- Y1: value 39MHz 10ppm -> 32MHz 7ppm
Other:
- note added: "PCB ANTENNA TUNING: US: C1=TBD, C2=TBD, C3=TBD EU: C1=TBD, C2=TBD, C3=TBD"
- note removed: "PCB ANTENNA TUNING: US: C4=TBD, C3=TBD, C4=TBD EU: C4=TBD, C3=TBD, C4=TBD"
Changed lines of the file:
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@@
 	(title_block
 		(title "ZRAD Mini Z-Wave Reference Application Design CZ20")
-		(date "2025-04-11")
+		(date "2025-05-13")
 		(rev "A1")
 		(company "Trident IoT")
@@
 		)
 	)
-	(text "PCB ANTENNA TUNING:\nUS: C4=TBD, C3=TBD, C4=TBD\nEU: C4=TBD, C3=TBD, C4=TBD"
+	(text "PCB ANTENNA TUNING:\nUS: C1=TBD, C2=TBD, C3=TBD\nEU: C1=TBD, C2=TBD, C3=TBD"
 		(exclude_from_sim no)
 		(at 198.882 83.058 0)
@@
 			)
 		)
-		(property "Value" "39MHz 10ppm"
+		(property "Value" "32MHz 7ppm"
 			(at 204.216 146.05 90)
 			(effects
@@
 			)
 		)
-		(property "Value" "100PF"
+		(property "Value" "120PF"
 			(at 243.205 88.265 0)
 			(effects
@@
 		(dnp no)
 		(property "Reference" "L8"
-			(at 142.24 92.71 90)
+			(at 139.954 98.298 90)
 			(effects
 				(font
@@
 			)
 		)
-		(property "Value" "4U7"
-			(at 142.24 97.155 90)
+		(property "Value" "4.7UH"
+			(at 142.24 95.758 90)
 			(effects
 				(font
@@
 			)
 		)
-		(property "Value" "100NF"
+		(property "Value" "100N"
 			(at 183.515 85.09 0)
 			(effects
@@
 			)
 		)
-		(property "Value" "47UH"
+		(property "Value" "47NH"
 			(at 236.855 82.55 90)
 			(effects
@@
 			)
 		)
-		(property "Value" "27UH"
+		(property "Value" "27NH"
 			(at 220.98 97.536 90)
 			(effects
@@
 			)
 		)
-		(property "Value" "8N5"
+		(property "Value" "8.5NH"
 			(at 228.346 111.506 90)
 			(effects
@@
 			)
 		)
-		(property "Value" "47UH"
+		(property "Value" "47NH"
 			(at 209.55 100.33 90)
 			(effects
@@
 			)
 		)
-		(property "Value" "27UH"
+		(property "Value" "27NH"
 			(at 209.55 104.14 90)
 			(effects
@@
 			)
 		)
-		(property "Value" "10UF"
-			(at 147.066 84.582 0)
+		(property "Value" "4U7"
+			(at 148.336 84.582 0)
 			(effects
 				(font
@@
 			)
 		)
-		(property "Value" "12N"
+		(property "Value" "12NH"
 			(at 236.22 111.76 90)
 			(effects
@@
 			)
 		)
-		(property "Footprint" "Capacitor_SMD:C_0603_1608Metric"
+		(property "Footprint" "Capacitor_SMD:C_0805_2012Metric"
 			(at 133.35 95.25 0)
 			(effects

Commit message: release ZRADTri Rev B
Parts:
- added R11: 1M, Resistor_SMD:R_0603_1608Metric, symbol Device:R_US
- added R12: NM, Resistor_SMD:R_0603_1608Metric, symbol Device:R_US
- D1: value QLSP14RGB_B -> BL-HJXGXBX32M-D; footprint ZReach:LED_QLSP14RGB -> LED_SMD:LED_Cree-PLCC4_3.2x2.8mm_CCW; symbol Device:LED_GRAB -> Device:LED_ARGB
- U1: footprint Package_DFN_QFN:TQFN-40-1EP_5x5mm_P0.4mm_EP3.5x3.5mm_ThermalVias -> Package_DFN_QFN:VQFN-40-1EP_5x5mm_P0.4mm_EP3.3x3.3mm
Connections:
- net +3.3V: now also D1.1 (A), R11.2; no longer D1.3 (A)
- net GND: now also R12.2
- net GP14: now also R11.1, R12.1
- net RFIN: no longer L4.1
- net RFIP: now also L4.1
- net at R2.1: now also D1.2 (RK); no longer D1.4 (BK)
- net at R3.1: now also D1.4 (BK); no longer D1.2 (RK)
- net at R1.1: now also D1.3 (GK); no longer D1.1 (GK)
Other:
- note added: "Hardware Version"
- note added: "PCB ANTENNA TUNING: US: C1=TBD, C2=TBD, C3=TBD EU: C1=TBD, C2=TBD, C3=TBD SMA Antenna: C1,C2,C3 NM"
- note removed: "PCB ANTENNA TUNING: US: C1=TBD, C2=TBD, C3=TBD EU: C1=TBD, C2=TBD, C3=TBD"
- moved on the sheet: R2, R3
